File: pcb/cnc-shield/cnc-shield.kicad_pcb (KiCad board)
At the start: 2 copper layers, 73 x 50 mm, 25 parts, among them J1 Servo, J2 A_STEPPER, J3 12V_BATTERY_SUPPLY, J4 B_STEPPER, J5 C_STEPPER, J6 Conn_02x05_Odd_Even, J7 5V_FROM_REGULATOR, U2 AMS1117-3.3

Commit message: added some pics
Other:
- net class +12V removed
- net class Default removed
