File: pcb/cnc_shield_mcu/cnc_shield_mcu.kicad_pcb (KiCad board)
At the start: 2 copper layers, 63 x 50 mm, 7 parts, among them J1 Conn_02x05_Odd_Even, U1 ESP32-DEV-30GPIO

Commit message: added some pics
Other:
- net class Default removed
